Commit message: add zylinder as collison geometry for wheels

File: models/curt_mini/robot.urdf.xacro (robot description, xacro)
@@ -49,7 +49,7 @@
     </visual>
     <collision>
-      <origin xyz="0 0 0" rpy="0 0 0" />
+      <origin xyz="0 0.01 0" rpy="${PI / 2} 0 0" />
       <geometry>
-        <mesh filename="file://$(arg path)/models/curt_mini/meshes/Wheel_01 .STL" />
+        <cylinder radius="${wheel_radius}" length="${wheel_width}"/>
       </geometry>
     </collision>
@@ -61,6 +61,7 @@
     <axis xyz="0 -1 0" />
     <dynamics damping="1.0" />
+    <limit effort="${max_effort}" velocity="${max_velocity}" />
   </joint>
-  <xacro:wheel_transmissions prefix="front_right" />
+  <xacro:wheel_transmissions prefix="front_right_motor" />
   <link name="front_left_wheel">
     <inertial>
@@ -79,7 +80,7 @@
     </visual>
     <collision>
-      <origin xyz="0 0 0" rpy="0 0 0" />
+      <origin xyz="0 -0.01 0" rpy="${PI / 2} 0 0" />
       <geometry>
-        <mesh filename="file://$(arg path)/models/curt_mini/meshes/Wheel_02.STL" />
+        <cylinder radius="${wheel_radius}" length="${wheel_width}"/>
       </geometry>
     </collision>
@@ -91,6 +92,7 @@
     <axis xyz="0 -1 0" />
     <dynamics damping="1.0" />
+    <limit effort="${max_effort}" velocity="${max_velocity}" />
   </joint>
-  <xacro:wheel_transmissions prefix="front_left" />
+  <xacro:wheel_transmissions prefix="front_left_motor" />
   <link name="back_right_wheel">
     <inertial>
@@ -109,7 +111,7 @@
     </visual>
     <collision>
-      <origin xyz="0 0 0" rpy="0 0 0" />
+      <origin xyz="0 0.01 0" rpy="${PI / 2} 0 0" />
       <geometry>
-        <mesh filename="file://$(arg path)/models/curt_mini/meshes/Wheel_03.STL" />
+        <cylinder radius="${wheel_radius}" length="${wheel_width}"/>
       </geometry>
     </collision>
@@ -121,6 +123,7 @@
     <axis xyz="0 -1 0" />
     <dynamics damping="1.0" />
+    <limit effort="${max_effort}" velocity="${max_velocity}" />
   </joint>
-  <xacro:wheel_transmissions prefix="back_right" />
+  <xacro:wheel_transmissions prefix="back_right_motor" />
   <link name="back_left_wheel">
     <inertial>
@@ -139,7 +142,7 @@
     </visual>
     <collision>
-      <origin xyz="0 0 0" rpy="0 0 0" />
+      <origin xyz="0 -0.01 0" rpy="${PI / 2} 0 0" />
       <geometry>
-        <mesh filename="file://$(arg path)/models/curt_mini/meshes/Wheel_04.STL" />
+        <cylinder radius="${wheel_radius}" length="${wheel_width}"/>
       </geometry>
     </collision>
@@ -151,6 +154,7 @@
     <axis xyz="0 -1 0" />
     <dynamics damping="1.0" />
+    <limit effort="${max_effort}" velocity="${max_velocity}" />
   </joint>
-  <xacro:wheel_transmissions prefix="back_left" />
+  <xacro:wheel_transmissions prefix="back_left_motor" />
   <!-- Import gazebo infos -->
   <xacro:if value="$(arg use_sim_time)" >
