Commit message: param changes for curt mini

File: models/curt_mini/gazebo.xacro (robot description, xacro)
@@ -8,4 +8,37 @@
     </plugin>
   </gazebo>
+  <!-- <gazebo>
+    <plugin name="joint_states" filename="libgazebo_ros_joint_state_publisher.so">
+      <joint_name>front_left_motor</joint_name>
+      <joint_name>front_right_motor</joint_name>
+      <joint_name>back_left_motor</joint_name>
+      <joint_name>back_right_motor</joint_name>
+    </plugin>
+  </gazebo>
+  <gazebo>
+    <plugin name='skid_steer_drive' filename='libgazebo_ros_diff_drive.so'>
+      <ros>
+        <remapping>cmd_vel:=/diff_drive_controller/cmd_vel_unstamped</remapping>
+        <remapping>odom:=wheel_odom</remapping>
+      </ros>
+      <num_wheel_pairs>2</num_wheel_pairs>
+      <left_joint>front_left_motor</left_joint>
+      <left_joint>back_left_motor</left_joint>
+      <right_joint>front_right_motor</right_joint>
+      <right_joint>back_right_motor</right_joint>
+      <wheel_separation>0.44</wheel_separation>
+      <wheel_separation>0.44</wheel_separation>
+      <wheel_diameter>0.26</wheel_diameter>
+      <wheel_diameter>0.26</wheel_diameter>
+      <max_wheel_torque>2000</max_wheel_torque>
+      <max_wheel_acceleration>10.0</max_wheel_acceleration>
+      <update_rate>500</update_rate>
+      <publish_odom>true</publish_odom>
+      <publish_odom_tf>true</publish_odom_tf>
+      <publish_wheel_tf>true</publish_wheel_tf>
+      <odometry_frame>odom</odometry_frame>
+      <robot_base_frame>base_link</robot_base_frame>
+    </plugin>
+  </gazebo> -->
   <gazebo reference="base_link">
     <material>Gazebo/Grey</material>

File: models/curt_mini/properties.xacro (robot description, xacro)
@@ -3,8 +3,13 @@
     <!-- Constants for robot -->
     <xacro:property name="PI" value="3.1415926535897931" />
+    <!-- robot limits -->
+    <xacro:property name="max_effort" value="50.0" />
+    <xacro:property name="max_velocity" value="5.0" />
+    <xacro:property name="wheel_radius" value="0.13" />
+    <xacro:property name="wheel_width" value="0.08" />
     <!-- Diff wheel ode params -->
     <xacro:macro name="wheel_ode_params">
-        <mu1 value="100" />
-        <mu2 value="0.2" />
+        <mu1 value="200" />
+        <mu2 value="0.3" />
         <kp value="10000000.0" />
         <kd value="1" />

Commit message: add depth camera sensor

File: models/curt_mini/gazebo.xacro (robot description, xacro)
@@ -134,3 +134,37 @@
     <material>Gazebo/Grey</material>
   </gazebo>
+  <gazebo reference="camera_link">
+    <sensor name="camera_link_camera" type="depth">
+      <always_on>true</always_on>
+      <update_rate>20</update_rate>
+      <pose>0 0 0 ${PI / 2} ${-PI / 2} 0</pose>
+      <camera name="realsense">
+        <horizontal_fov>1.047198</horizontal_fov>
+        <image>
+          <width>640</width>
+          <height>480</height>
+          <format>RGB8</format>
+        </image>
+        <clip>
+          <near>0.05</near>
+          <far>5</far>
+        </clip>
+      </camera>
+      <plugin name="camera_link_controller" filename="libgazebo_ros_camera.so">
+        <ros>
+          <namespace>d430</namespace>
+          <remapping>camera/image_raw:=color/image_raw</remapping>
+          <remapping>camera/depth/image_raw:=depth/image_rect_raw</remapping>
+          <remapping>camera/camera_info:=camera_info</remapping>
+          <remapping>camera/depth/camera_info:=depth/camera_info</remapping>
+          <remapping>camera/points:=depth/points</remapping>
+        </ros>
+        <camera_name>camera</camera_name>
+        <frame_name>camera_link</frame_name>
+        <hack_baseline>0.07</hack_baseline>
+        <min_depth>0.05</min_depth>
+        <max_depth>8.0</max_depth>
+      </plugin>
+    </sensor>
+  </gazebo>
 </robot>

File: models/curt_mini/sensors.xacro (robot description, xacro)
@@ -17,4 +17,19 @@
   </joint>
   <link name="gps_link" />
+  <!-- Camera -->
+  <joint name="base_link_to_camera" type="fixed">
+    <parent link="base_link" />
+    <child link="camera_link" />
+    <origin xyz="0.0 0.0 0.7" rpy="${-PI / 2 - PI / 6} 0.0 ${-PI / 2}" />
+  </joint>
+  <link name="camera_link" >
+    <visual>
+      <origin rpy="0.0 0.0 0.0" xyz="0 0 0" />
+      <geometry>
+          <box size="0.10 0.05 0.05" />
+      </geometry>
+      <material name="grey" />
+  </visual>
+  </link>
   <!-- Velodyne -->
   <xacro:VLP-16 parent="base_link" name="velodyne" topic="/lidar_points" organize_cloud="false" hz="10" samples="440" gpu="false">
