Commit message: better values for sensor positions in urdf

File: models/curt_mini/sensors.xacro (robot description, xacro)
@@ -14,10 +14,10 @@
     <parent link="base_link" />
     <child link="gps_link" />
-    <origin xyz="0.0 0.0 0.0" />
+    <origin xyz="-0.14 0.0 0.34" />
   </joint>
   <link name="gps_link" />
   <!-- Velodyne -->
   <xacro:VLP-16 parent="base_link" name="velodyne" topic="/lidar_points" organize_cloud="false" hz="10" samples="440" gpu="false">
-    <origin xyz="0.25 0.0 0.2" rpy="0 ${PI / 8} 0" />
+    <origin xyz="0.175 0.0 0.31" rpy="0 ${PI / 12} 0" />
   </xacro:VLP-16>
 </robot>

Commit message: collision_avoidance params and traversability map in costmap

File: models/curt_mini/sensors.xacro (robot description, xacro)
@@ -34,6 +34,7 @@
   </visual>
   </link>
+  <!-- <xacro:macro name="VLP-16" params="*origin parent:=base_link name:=velodyne tf_prefix:='' topic:=/velodyne_points organize_cloud:=false hz:=10 lasers:=16 samples:=1875 collision_range:=0.3 min_range:=0.9 max_range:=130.0 noise:=0.008 min_angle:=-${M_PI} max_angle:=${M_PI} gpu:=false"> -->
   <!-- Velodyne -->
-  <xacro:VLP-16 parent="base_link" name="velodyne" topic="/lidar_points" organize_cloud="false" hz="10" samples="440" gpu="false">
+  <xacro:VLP-16 parent="base_link" name="velodyne" min_range="0.1" topic="/lidar_points" organize_cloud="false" hz="10" samples="440" gpu="false">
     <origin xyz="0.175 0.0 0.31" rpy="0 ${PI / 12} 0" />
   </xacro:VLP-16>

Commit message: Agritechnica setup

File: models/curt_mini/sensors.xacro (robot description, xacro)
@@ -36,6 +36,6 @@
   <!-- <xacro:macro name="VLP-16" params="*origin parent:=base_link name:=velodyne tf_prefix:='' topic:=/velodyne_points organize_cloud:=false hz:=10 lasers:=16 samples:=1875 collision_range:=0.3 min_range:=0.9 max_range:=130.0 noise:=0.008 min_angle:=-${M_PI} max_angle:=${M_PI} gpu:=false"> -->
   <!-- Velodyne -->
-  <xacro:VLP-16 parent="base_link" name="velodyne" min_range="0.1" topic="/lidar_points" organize_cloud="false" hz="10" samples="440" gpu="false">
-    <origin xyz="0.175 0.0 0.31" rpy="0 ${PI / 12} 0" />
+  <xacro:VLP-16 parent="base_link" name="velodyne" topic="/lidar_points" organize_cloud="false" hz="10" samples="440" gpu="false">
+    <origin xyz="0.175 0.0 0.31" rpy="0 0 ${PI}" />
   </xacro:VLP-16>
 </robot>

Commit message: Updated urdf and nav startup

File: models/curt_mini/sensors.xacro (robot description, xacro)
@@ -9,5 +9,5 @@
     <parent link="base_link" />
     <child link="imu_link" />
-    <origin xyz="0.0 0.0 0.0" />
+    <origin xyz="0.035 0.03 0.12" rpy="0.0 3.14159 0.0"/>
   </joint>
   <link name="imu_link" />
@@ -23,5 +23,5 @@
     <parent link="base_link" />
     <child link="camera_link" />
-    <origin xyz="0.0 0.0 0.7" rpy="${-PI / 2 - PI / 6} 0.0 ${-PI / 2}" />
+    <origin xyz="0.32 0.02 0.18" rpy="0.0 0.2792 0.0" /> <!-- 16° down -->
   </joint>
   <link name="camera_link" >
@@ -34,8 +34,18 @@
   </visual>
   </link>
+  <!-- lidar -->
+  <joint name="base_link_to_lidar" type="fixed">
+    <parent link="base_link" />
+    <child link="lidar_link" />
+    <origin xyz="0.2 0.0 0.4" rpy="0 0 0" />
+  </joint>
+  <link name="lidar_link" />
+  <xacro:VLP-16 parent="lidar_link" name="velodyne" topic="/ouster/points" organize_cloud="false" min_range="0.1" hz="10" samples="1875" gpu="true">
+    <origin xyz="0.0 0.0 0.0" rpy="0 0 0" />
+  </xacro:VLP-16>
   <!-- <xacro:macro name="VLP-16" params="*origin parent:=base_link name:=velodyne tf_prefix:='' topic:=/velodyne_points organize_cloud:=false hz:=10 lasers:=16 samples:=1875 collision_range:=0.3 min_range:=0.9 max_range:=130.0 noise:=0.008 min_angle:=-${M_PI} max_angle:=${M_PI} gpu:=false"> -->
-  <!-- Velodyne -->
+  <!-- Velodyne
   <xacro:VLP-16 parent="base_link" name="velodyne" topic="/lidar_points" organize_cloud="false" hz="10" samples="440" gpu="false">
     <origin xyz="0.175 0.0 0.31" rpy="0 0 ${PI}" />
-  </xacro:VLP-16>
+  </xacro:VLP-16> -->
 </robot>

Commit message: add lpms-al3 imu

File: models/curt_mini/sensors.xacro (robot description, xacro)
@@ -5,9 +5,10 @@
   <!-- Some properties -->
   <xacro:include filename="$(find curt_mini)/models/curt_mini/properties.xacro" />
-  <!-- IMU -->
+  <!-- LPResearch CANAL3 IMU -->
   <joint name="base_link_to_imu" type="fixed">
     <parent link="base_link" />
     <child link="imu_link" />
-    <origin xyz="0.035 0.03 0.12" rpy="0.0 3.14159 0.0"/>
+    <!-- Position roughly estimated -->
+    <origin xyz="0.0 -0.03 0.14" rpy="0.0 0.0 ${pi/2}"/>
   </joint>
   <link name="imu_link" />

Commit message: restore xsens config as comments

File: models/curt_mini/sensors.xacro (robot description, xacro)
@@ -5,4 +5,10 @@
   <!-- Some properties -->
   <xacro:include filename="$(find curt_mini)/models/curt_mini/properties.xacro" />
+  <!-- Xsens IMU -->
+  <!-- <joint name="base_link_to_imu" type="fixed">
+    <parent link="base_link" />
+    <child link="imu_link" />
+    <origin xyz="0.035 0.03 0.12" rpy="0.0 3.14159 0.0"/>
+  </joint> -->
   <!-- LPResearch CANAL3 IMU -->
   <joint name="base_link_to_imu" type="fixed">

Commit message: add basic livox sensor setup

File: models/curt_mini/sensors.xacro (robot description, xacro)
@@ -87,3 +87,11 @@
     <origin xyz="0.175 0.0 0.31" rpy="0 0 ${PI}" />
   </xacro:VLP-16> -->
+  <!-- Livox MID-70 LiDAR -->
+  <!-- Preliminary mount, to be changed once a proper mount is fabricated -->
+  <joint name="base_link_to_livox" type="fixed">
+    <parent link="base_link" />
+    <child link="livox" />
+    <origin xyz="0.2 0.0 0.3" rpy="${pi} 0 0" />
+  </joint>
+  <link name="livox" />
 </robot>

Commit message: Added Robosense RS16 Lidar

File: models/curt_mini/sensors.xacro (robot description, xacro)
@@ -41,5 +41,12 @@
   </visual>
   </link>
-  <!-- lidar -->
+  <!-- lidar robosense -->
+  <joint name="base_link_to_lidar" type="fixed">
+    <parent link="base_link" />
+    <child link="lidar_link" />
+    <origin xyz="0.215 0.0 0.4" rpy="0 0 0" />
+  </joint>
+  <link name="lidar_link" />
+  <!-- lidar ouster
   <joint name="base_link_to_lidar" type="fixed">
     <parent link="base_link" />
@@ -48,4 +55,5 @@
   </joint>
   <link name="lidar_link" />
+  -->
   <gazebo reference="lidar_link">
     <sensor name='gpu_lidar' type='gpu_lidar'>

Commit message: livox mounting

File: models/curt_mini/sensors.xacro (robot description, xacro)
@@ -95,10 +95,19 @@
     <origin xyz="0.175 0.0 0.31" rpy="0 0 ${PI}" />
   </xacro:VLP-16> -->
-  <!-- Livox MID-70 LiDAR -->
-  <!-- Preliminary mount, to be changed once a proper mount is fabricated -->
+  <!-- livox mid-70 lidar -->
+  <!-- Mounted with 3D printed mounting adapter centered in Y-direction and as far forward as
+  possible on the robot -->
+  <!-- front bottom edge of housing -->
   <joint name="base_link_to_livox" type="fixed">
     <parent link="base_link" />
+    <child link="livox_housing" />
+    <origin xyz="0.268 0.0 0.25" rpy="0 0 0" />
+  </joint>
+  <link name="livox_housing" />
+  <!-- livox sensor frame -->
+  <joint name="livox_internal_offset" type="fixed">
+    <parent link="livox_housing" />
     <child link="livox" />
-    <origin xyz="0.2 0.0 0.3" rpy="${pi} 0 0" />
+    <origin xyz="-0.0162 0.0 0.0324" rpy="0 0 0" />
   </joint>
   <link name="livox" />
