Commit message: remove more unused config files

File: curt_mini/models/curt_mini/gazebo.xacro (robot description, xacro)
@@ -72,5 +72,5 @@
         <ros>
           <namespace>imu</namespace>
-          <remapping>~/out:=data_raw</remapping>
+          <remapping>~/out:=data</remapping>
         </ros>
         <initial_orientation_as_reference>false</initial_orientation_as_reference>
@@ -78,55 +78,4 @@
     </sensor>
   </gazebo>
-  <!-- GPS -->
-  <gazebo reference="gps_link">
-    <sensor name="gps_sensor" type="gps">
-      <always_on>true</always_on>
-      <update_rate>1.0</update_rate>
-      <plugin name="gps_controller" filename="libgazebo_ros_gps_sensor.so">
-        <ros>
-          <!-- <namespace>/br</namespace> -->
-          <remapping>gps_controller/out:=gps/fix</remapping>
-        </ros>
-        <frame_name>gps_link</frame_name>
-      </plugin>
-    </sensor>
-    <material>Gazebo/Grey</material>
-  </gazebo>
-<!--
-  <gazebo reference="camera_link">
-    <sensor name="camera_link_camera" type="depth">
-      <always_on>true</always_on>
-      <update_rate>20</update_rate>
-      <camera name="realsense">
-        <pose>0 0 0 ${PI / 2} ${-PI / 2} 0</pose>
-        <horizontal_fov>1.047198</horizontal_fov>
-        <image>
-          <width>640</width>
-          <height>480</height>
-          <format>RGB8</format>
-        </image>
-        <clip>
-          <near>0.05</near>
-          <far>5</far>
-        </clip>
-      </camera>
-      <plugin name="camera_link_controller" filename="libgazebo_ros_camera.so">
-        <ros>
-          <namespace>d430</namespace>
-          <remapping>camera/image_raw:=color/image_raw</remapping>
-          <remapping>camera/depth/image_raw:=depth/image_rect_raw</remapping>
-          <remapping>camera/camera_info:=camera_info</remapping>
-          <remapping>camera/depth/camera_info:=depth/camera_info</remapping>
-          <remapping>camera/points:=depth/points</remapping>
-        </ros>
-        <camera_name>camera</camera_name>
-        <frame_name>camera_link</frame_name>
-        <hack_baseline>0.07</hack_baseline>
-        <min_depth>0.05</min_depth>
-        <max_depth>8.0</max_depth>
-      </plugin>
-    </sensor>
-  </gazebo>
--->
   <gazebo>
     <plugin filename="gz-sim-pose-publisher-system" name="gz::sim::systems::PosePublisher">
