Commit message: remove unused sensor links

File: curt_mini/models/curt_mini/sensors.xacro (robot description, xacro)
@@ -1,14 +1,6 @@
 <?xml version="1.0"?>
 <robot xmlns:xacro="http://www.ros.org/wiki/xacro">
-  <!-- Package to load velodyne sensor
-  <xacro:include filename="$(find velodyne_description)/urdf/VLP-16.urdf.xacro" /-->
   <!-- Some properties -->
   <xacro:include filename="$(find curt_mini)/models/curt_mini/properties.xacro" />
-  <!-- Xsens IMU -->
-  <!-- <joint name="base_link_to_imu" type="fixed">
-    <parent link="base_link" />
-    <child link="imu_link" />
-    <origin xyz="0.035 0.03 0.12" rpy="0.0 3.14159 0.0"/>
-  </joint> -->
   <!-- LPResearch CANAL3 IMU -->
   <joint name="base_link_to_imu" type="fixed">
@@ -19,96 +11,3 @@
   </joint>
   <link name="imu_link" />
-  <!-- GPS -->
-  <joint name="base_link_to_gps" type="fixed">
-    <parent link="base_link" />
-    <child link="gps_link" />
-    <origin xyz="-0.14 0.0 0.34" />
-  </joint>
-  <link name="gps_link" />
-  <!-- Camera -->
-  <joint name="base_link_to_camera" type="fixed">
-    <parent link="base_link" />
-    <child link="camera_link" />
-    <origin xyz="0.32 0.02 0.18" rpy="0.0 0.2792 0.0" /> <!-- 16° down -->
-  </joint>
-  <link name="camera_link" >
-    <visual>
-      <origin rpy="0.0 0.0 0.0" xyz="0 0 0" />
-      <geometry>
-          <box size="0.10 0.05 0.05" />
-      </geometry>
-      <material name="grey" />
-  </visual>
-  </link>
-  <!-- lidar robosense -->
-  <joint name="base_link_to_lidar" type="fixed">
-    <parent link="base_link" />
-    <child link="lidar_link" />
-    <origin xyz="0.215 0.0 0.4" rpy="0 0 0" />
-  </joint>
-  <link name="lidar_link" />
-  <!-- lidar ouster
-  <joint name="base_link_to_lidar" type="fixed">
-    <parent link="base_link" />
-    <child link="lidar_link" />
-    <origin xyz="0.2 0.0 0.4" rpy="0 0 0" />
-  </joint>
-  <link name="lidar_link" />
-  -->
-  <gazebo reference="lidar_link">
-    <sensor name='gpu_lidar' type='gpu_lidar'>
-      <gz_frame_id>lidar_link</gz_frame_id>
-      <topic>lidar</topic>
-      <update_rate>20</update_rate>
-      <ray>
-        <scan>
-          <horizontal>
-            <samples>1024</samples>
-            <resolution>1</resolution>
-            <min_angle>${-pi}</min_angle>
-            <max_angle>${pi}</max_angle>
-          </horizontal>
-          <vertical>
-            <samples>32</samples>
-            <resolution>1</resolution>
-            <min_angle>${-pi/4}</min_angle>
-            <max_angle>${pi/4}</max_angle>
-          </vertical>
-        </scan>
-        <range>
-          <min>0.5</min>
-          <max>35.0</max>
-        </range>
-      </ray>
-      <always_on>1</always_on>
-      <visualize>true</visualize>
-    </sensor>
-  </gazebo>
-<!--
-  <xacro:VLP-16 parent="lidar_link" name="velodyne" topic="/ouster/points" organize_cloud="false" min_range="0.1" hz="10" samples="1875" gpu="true">
-    <origin xyz="0.0 0.0 0.0" rpy="0 0 0" />
-  </xacro:VLP-16>
--->
-  <!-- <xacro:macro name="VLP-16" params="*origin parent:=base_link name:=velodyne tf_prefix:='' topic:=/velodyne_points organize_cloud:=false hz:=10 lasers:=16 samples:=1875 collision_range:=0.3 min_range:=0.9 max_range:=130.0 noise:=0.008 min_angle:=-${M_PI} max_angle:=${M_PI} gpu:=false"> -->
-  <!-- Velodyne
-  <xacro:VLP-16 parent="base_link" name="velodyne" topic="/lidar_points" organize_cloud="false" hz="10" samples="440" gpu="false">
-    <origin xyz="0.175 0.0 0.31" rpy="0 0 ${PI}" />
-  </xacro:VLP-16> -->
-  <!-- livox mid-70 lidar -->
-  <!-- Mounted with 3D printed mounting adapter centered in Y-direction and as far forward as
-  possible on the robot -->
-  <!-- front bottom edge of housing -->
-  <joint name="base_link_to_livox" type="fixed">
-    <parent link="base_link" />
-    <child link="livox_housing" />
-    <origin xyz="0.268 0.0 0.25" rpy="0 0 0" />
-  </joint>
-  <link name="livox_housing" />
-  <!-- livox sensor frame -->
-  <joint name="livox_internal_offset" type="fixed">
-    <parent link="livox_housing" />
-    <child link="livox" />
-    <origin xyz="-0.0162 0.0 0.0324" rpy="0 0 0" />
-  </joint>
-  <link name="livox" />
 </robot>

Commit message: rough configuration of new imu position

File: curt_mini/models/curt_mini/sensors.xacro (robot description, xacro)
@@ -7,6 +7,6 @@
     <parent link="base_link" />
     <child link="imu_link" />
-    <!-- Position roughly estimated -->
-    <origin xyz="0.0 -0.03 0.14" rpy="0.0 0.0 ${pi/2}"/>
+    <!-- TODO: Verify new IMU mounting -->
+    <origin xyz="0.1 0.0 0.015" rpy="0.0 0.0 ${pi/2}"/>
   </joint>
   <link name="imu_link" />

Commit message: configure IMU position from CAD model

File: curt_mini/models/curt_mini/sensors.xacro (robot description, xacro)
@@ -7,6 +7,5 @@
     <parent link="base_link" />
     <child link="imu_link" />
-    <!-- TODO: Verify new IMU mounting -->
-    <origin xyz="0.1 0.0 0.015" rpy="0.0 0.0 ${pi/2}"/>
+    <origin xyz="0.062 0.0 0.015" rpy="0.0 0.0 ${pi/2}"/>
   </joint>
   <link name="imu_link" />
