Commit message: cherry pick wheel velocity limit fix for ros kilted

File: curt_mini/models/curt_mini/properties.xacro (robot description, xacro)
@@ -5,5 +5,6 @@
     <!-- robot limits -->
     <xacro:property name="max_effort" value="50.0" />
-    <xacro:property name="max_velocity" value="5.0" />
+    <!-- joint limit for wheels, radian/second -->
+    <xacro:property name="max_velocity" value="20.0" />
     <xacro:property name="wheel_radius" value="0.13" />
     <xacro:property name="wheel_width" value="0.08" />

File: curt_mini/models/curt_mini/robot.urdf.xacro (robot description, xacro)
@@ -62,5 +62,5 @@
     <axis xyz="0 -1 0" />
     <dynamics damping="1.0" />
-    <limit effort="${max_effort}" velocity="${max_velocity}" />
+    <limit effort="${max_effort}" velocity="${max_wheel_velocity}" />
   </joint>
   <xacro:wheel_transmissions prefix="front_right_motor" />
@@ -93,5 +93,5 @@
     <axis xyz="0 -1 0" />
     <dynamics damping="1.0" />
-    <limit effort="${max_effort}" velocity="${max_velocity}" />
+    <limit effort="${max_effort}" velocity="${max_wheel_velocity}" />
   </joint>
   <xacro:wheel_transmissions prefix="front_left_motor" />
@@ -124,5 +124,5 @@
     <axis xyz="0 -1 0" />
     <dynamics damping="1.0" />
-    <limit effort="${max_effort}" velocity="${max_velocity}" />
+    <limit effort="${max_effort}" velocity="${max_wheel_velocity}" />
   </joint>
   <xacro:wheel_transmissions prefix="back_right_motor" />
@@ -155,5 +155,5 @@
     <axis xyz="0 -1 0" />
     <dynamics damping="1.0" />
-    <limit effort="${max_effort}" velocity="${max_velocity}" />
+    <limit effort="${max_effort}" velocity="${max_wheel_velocity}" />
   </joint>
   <xacro:wheel_transmissions prefix="back_left_motor" />

Commit message: fix max_wheel_velocity

File: curt_mini/models/curt_mini/properties.xacro (robot description, xacro)
@@ -6,5 +6,5 @@
     <xacro:property name="max_effort" value="50.0" />
     <!-- joint limit for wheels, radian/second -->
-    <xacro:property name="max_velocity" value="20.0" />
+    <xacro:property name="max_wheel_velocity" value="20.0" />
     <xacro:property name="wheel_radius" value="0.13" />
     <xacro:property name="wheel_width" value="0.08" />

Commit message: update URDF and meshes

File: curt_mini/models/curt_mini/properties.xacro (robot description, xacro)
@@ -17,15 +17,3 @@
         <fdir1 value="1 0 0" />
     </xacro:macro>
-    <!-- transmissions -->
-    <xacro:macro name="wheel_transmissions" params="prefix">
-        <transmission name="${prefix}_wheel_trans">
-            <type>transmission_interface/SimpleTransmission</type>
-            <joint name="${prefix}">
-              <hardwareInterface>hardware_interface/VelocityJointInterface</hardwareInterface>
-            </joint>
-            <actuator name="${prefix}_wheel_actuator">
-              <mechanicalReduction>1</mechanicalReduction>
-            </actuator>
-          </transmission>
-    </xacro:macro>
 </robot>

File: curt_mini/models/curt_mini/robot.urdf.xacro (robot description, xacro)
@@ -13,11 +13,12 @@
   <xacro:include filename="$(find curt_mini)/models/curt_mini/sensors.xacro" />
   <link name="base_link" />
-  <!-- Chassis link at same position as base_link, as root is not allowed to have inertial information -->
+  <!-- Chassis link at same position as base_link, as root is not allowed to have inertial
+  information -->
   <link name="chassis">
     <inertial>
-      <origin xyz="-0.0076959 -0.0021447 0.056616" rpy="0 0 0" />
-      <mass value="9.6512" />
-      <inertia ixx="0.036046" ixy="-1.6181E-05" ixz="-0.00088314" iyy="0.10986" iyz="-3.4695E-06"
-        izz="0.12533" />
+      <origin xyz="0.011876 0.003999 0.048645" rpy="0 0 0" />
+      <mass value="9.0318" />
+      <inertia ixx="0.04558" ixy="-2.4654E-05" ixz="0.0014869" iyy="0.059986" iyz="2.4934E-05"
+        izz="0.09132" />
     </inertial>
     <visual>
@@ -27,5 +28,5 @@
       </geometry>
       <material name="">
-        <color rgba="0.5098 0.5098 0.54902 1" />
+        <color rgba="0.79216 0.81961 0.93333 1" />
       </material>
     </visual>
@@ -37,5 +38,5 @@
     </collision>
   </link>
-  <joint name="base_to_footprint" type="fixed">
+  <joint name="base_to_chassis" type="fixed">
     <parent link="base_link" />
     <child link="chassis" />
@@ -43,16 +44,16 @@
   <link name="front_right_wheel">
     <inertial>
-      <origin xyz="-5.87030424270552E-15 0.00750997550383756 -5.38805111638396E-15" rpy="0 0 0" />
-      <mass value="1.16081815267191" />
-      <inertia ixx="0.00489876810873934" ixy="9.50165704321153E-19" ixz="-2.61848606081355E-08"
-        iyy="0.00918238967794609" iyz="-1.71449040958554E-17" izz="0.00489885881575725" />
+      <origin xyz="-2.8086E-05 0.013016 2.8089E-05" rpy="0 0 0" />
+      <mass value="0.61321" />
+      <inertia ixx="0.0031957" ixy="-6.9366E-08" ixz="-8.7949E-07" iyy="0.0057902" iyz="6.9371E-08"
+        izz="0.0031957" />
     </inertial>
     <visual>
       <origin xyz="0 0 0" rpy="0 0 0" />
       <geometry>
-        <mesh filename="file://$(arg path)/models/curt_mini/meshes/Wheel_01 .STL" />
+        <mesh filename="file://$(arg path)/models/curt_mini/meshes/wheel4_link.STL" />
       </geometry>
       <material name="">
-        <color rgba="0.298039215686275 0.298039215686275 0.298039215686275 1" />
+        <color rgba="0.79216 0.81961 0.93333 1" />
       </material>
     </visual>
@@ -65,26 +66,25 @@
   </link>
   <joint name="front_right_motor" type="continuous">
-    <origin xyz="0.259999999999997 -0.2140000002693 -0.0264914703891407" rpy="3.14159265358979 0 0" />
+    <origin xyz="0.25995 -0.258 -0.030204" rpy="0 0 0" />
     <parent link="base_link" />
     <child link="front_right_wheel" />
-    <axis xyz="0 -1 0" />
+    <axis xyz="0 1 0" />
     <dynamics damping="1.0" />
     <limit effort="${max_effort}" velocity="${max_wheel_velocity}" />
   </joint>
-  <xacro:wheel_transmissions prefix="front_right_motor" />
   <link name="front_left_wheel">
     <inertial>
-      <origin xyz="2.97539770599542E-14 -0.00750997550383714 6.53053999766229E-14" rpy="0 0 0" />
-      <mass value="1.16081815267191" />
-      <inertia ixx="0.00489876810873935" ixy="3.91724337570418E-19" ixz="2.61848606067545E-08"
-        iyy="0.00918238967794612" iyz="1.81861039773823E-17" izz="0.00489885881575728" />
+      <origin xyz="2.8086E-05 -0.013016 2.8089E-05" rpy="0 0 0" />
+      <mass value="0.61321" />
+      <inertia ixx="0.0031957" ixy="-6.9366E-08" ixz="8.7949E-07" iyy="0.0057902" iyz="-6.9371E-08"
+        izz="0.0031957" />
     </inertial>
     <visual>
       <origin xyz="0 0 0" rpy="0 0 0" />
       <geometry>
-        <mesh filename="file://$(arg path)/models/curt_mini/meshes/Wheel_02.STL" />
+        <mesh filename="file://$(arg path)/models/curt_mini/meshes/wheel1_link.STL" />
       </geometry>
       <material name="">
-        <color rgba="0.298039215686275 0.298039215686275 0.298039215686275 1" />
+        <color rgba="0.79216 0.81961 0.93333 1" />
       </material>
     </visual>
@@ -97,26 +97,25 @@
   </link>
   <joint name="front_left_motor" type="continuous">
-    <origin xyz="0.259999999999997 0.2140000002693 -0.0264914703891414" rpy="3.14159265358979 0 0" />
+    <origin xyz="0.25995 0.258 -0.030204" rpy="0 0 0" />
     <parent link="base_link" />
     <child link="front_left_wheel" />
-    <axis xyz="0 -1 0" />
+    <axis xyz="0 1 0" />
     <dynamics damping="1.0" />
     <limit effort="${max_effort}" velocity="${max_wheel_velocity}" />
   </joint>
-  <xacro:wheel_transmissions prefix="front_left_motor" />
   <link name="back_right_wheel">
     <inertial>
-      <origin xyz="-3.25850457727483E-14 0.00750997550383728 5.8935495372836E-14" rpy="0 0 0" />
-      <mass value="1.16081815267191" />
-      <inertia ixx="0.00489876810873933" ixy="9.33801693307905E-19" ixz="-2.61848606033406E-08"
-        iyy="0.00918238967794609" iyz="-1.82258288287945E-17" izz="0.00489885881575725" />
+      <origin xyz="-2.8086E-05 0.013016 2.8089E-05" rpy="0 0 0" />
+      <mass value="0.61321" />
+      <inertia ixx="0.0031957" ixy="-6.9366E-08" ixz="-8.7949E-07" iyy="0.0057902" iyz="6.9371E-08"
+        izz="0.0031957" />
     </inertial>
     <visual>
       <origin xyz="0 0 0" rpy="0 0 0" />
       <geometry>
-        <mesh filename="file://$(arg path)/models/curt_mini/meshes/Wheel_03.STL" />
+        <mesh filename="file://$(arg path)/models/curt_mini/meshes/wheel3_link.STL" />
       </geometry>
       <material name="">
-        <color rgba="1 1 1 1" />
+        <color rgba="0.79216 0.81961 0.93333 1" />
       </material>
     </visual>
@@ -129,26 +128,25 @@
   </link>
   <joint name="back_right_motor" type="continuous">
-    <origin xyz="-0.259999999999997 -0.214000000269301 -0.02649147038914" rpy="3.14159265358979 0 0" />
+    <origin xyz="-0.26 -0.258 -0.022755" rpy="0 0 0" />
     <parent link="base_link" />
     <child link="back_right_wheel" />
-    <axis xyz="0 -1 0" />
+    <axis xyz="0 1 0" />
     <dynamics damping="1.0" />
     <limit effort="${max_effort}" velocity="${max_wheel_velocity}" />
   </joint>
-  <xacro:wheel_transmissions prefix="back_right_motor" />
   <link name="back_left_wheel">
     <inertial>
-      <origin xyz="3.05311331771918E-15 -0.00750997550383753 2.26554885962571E-15" rpy="0 0 0" />
-      <mass value="1.16081815267191" />
-      <inertia ixx="0.00489876810873933" ixy="1.74686590365548E-18" ixz="2.61848606031113E-08"
-        iyy="0.00918238967794607" iyz="1.56928180377104E-17" izz="0.00489885881575724" />
+      <origin xyz="2.8086E-05 -0.013016 2.8089E-05" rpy="0 0 0" />
+      <mass value="0.61321" />
+      <inertia ixx="0.0031957" ixy="-6.9366E-08" ixz="8.7949E-07" iyy="0.0057902" iyz="-6.9371E-08"
+        izz="0.0031957" />
     </inertial>
     <visual>
       <origin xyz="0 0 0" rpy="0 0 0" />
       <geometry>
-        <mesh filename="file://$(arg path)/models/curt_mini/meshes/Wheel_04.STL" />
+        <mesh filename="file://$(arg path)/models/curt_mini/meshes/wheel2_link.STL" />
       </geometry>
       <material name="">
-        <color rgba="0.298039215686275 0.298039215686275 0.298039215686275 1" />
+        <color rgba="0.79216 0.81961 0.93333 1" />
       </material>
     </visual>
@@ -161,12 +159,11 @@
   </link>
   <joint name="back_left_motor" type="continuous">
-    <origin xyz="-0.259999999999997 0.2140000002693 -0.0264914703891408" rpy="3.14159265358979 0 0" />
+    <origin xyz="-0.26 0.258 -0.022755" rpy="0 0 0" />
     <parent link="base_link" />
     <child link="back_left_wheel" />
-    <axis xyz="0 -1 0" />
+    <axis xyz="0 1 0" />
     <dynamics damping="1.0" />
     <limit effort="${max_effort}" velocity="${max_wheel_velocity}" />
   </joint>
-  <xacro:wheel_transmissions prefix="back_left_motor" />
   <!-- Import gazebo infos -->
   <xacro:if value="$(arg simulation)">
